Commit message: feat: add LinkerForce MuJoCo retarget mappings

File: src/linkerhand_retarget/linkerhand_retarget/assets/robots/hands/linker_hand/o20_left/linkerhand_o20_left.urdf (robot description, URDF)
Before this commit: robot linkerhand_o20_left.urdf, 22 links, 21 joints
Links:
- removed link index_proximal
- removed link middle_proximal
- removed link pinky_proximal
- removed link ring_proximal
- removed link thumb_metacarpals
- link hand_base_link: mass 0.110373495507463 -> 0.0657305134785705
- link index_distal: mass 0.00334170259772608 -> 0.004003
- link index_metacarpals: mass 0.000895516429792169 -> 0.0072705
- link index_middle: mass 0.00237827499847615 -> 0.0083271
- link middle_distal: mass 0.00334170288968694 -> 0.00400304702685047
- link middle_metacarpals: mass 0.000895516947435045 -> 0.00727048835691936
- link middle_middle: mass 0.00237827502274046 -> 0.00832707181666394
- link pinky_distal: mass 0.00334170283969146 -> 0.00400304621179198
- link pinky_metacarpals: mass 0.000895516947513541 -> 0
- link pinky_middle: mass 0.00237827431921004 -> 0.00832713433907816
- link ring_distal: mass 0.00334170280386792 -> 0.00400304721195506
- link ring_metacarpals: mass 0.000895516612684195 -> 0.0072704883571626
- link ring_middle: mass 0.00237827433282015 -> 0.00832712852462523
- link thumb_distal: mass 0.00382046638843239 -> 0.00884959085475471
- link thumb_metacarpals_base1: mass 0.0160351802817401 -> 0.00792340800041424
- link thumb_metacarpals_base2: mass 0.00183264554882498 -> 0.00201755096384541
- link thumb_proximal: mass 0.00549015507433734 -> 0.00586560783329691
Joints:
- removed joint index_mcp_pitch
- removed joint middle_mcp_pitch
- removed joint pinky_mcp_pitch
- removed joint ring_mcp_pitch
- removed joint thumb_cmc_pitch
- removed joint thumb_ip
- added joint thumb_dip: type revolute, parent thumb_proximal, child thumb_distal, origin xyz=0.0496008878156415 0.00064670858859911 0.01200524971208 rpy=0 0 0, axis 0.013038356643959 -0.999914997015258 0, limit lower=0 upper=1.5568 effort=0 velocity=0
- joint index_dip: axis 0 1 0 -> 0 1 1.7355E-05; limit lower=0 upper=1.55 effort=100 velocity=1 -> lower=0 upper=1.9897 effort=0 velocity=0; mimic joint=index_pip multiplier=0.89 offset=0 -> (none); origin xyz=0.0028245 0 0.031696 rpy=0 0 0 -> xyz=0.00032142 0 0.047999 rpy=0 0 0
- joint index_mcp_roll: axis 1 0 0 -> 0.99996 -0.0088916 0; limit lower=-0.23 upper=0.23 effort=100 velocity=1 -> lower=-0.08726 upper=0.3543 effort=0 velocity=0; origin xyz=0.0038 -0.03525 0.1481 rpy=0 0 0 -> xyz=-0.0024054 -0.032129 0.095682 rpy=0 0 0
- joint index_pip: axis 0 1 0 -> 0 1 1.3016E-05; limit lower=0 upper=1.74 effort=100 velocity=1 -> lower=0 upper=1.9548 effort=0 velocity=0; origin xyz=-0.0041946 0 0.044819 rpy=0 0 0 -> xyz=0.014909 0 0.0135 rpy=0 0 0; parent index_proximal -> index_metacarpals
- joint middle_dip: axis 0 1 0 -> 0 1 1.7355E-05; limit lower=0 upper=1.55 effort=100 velocity=1 -> lower=0 upper=1.9897 effort=0 velocity=0; mimic joint=middle_pip multiplier=0.89 offset=0 -> (none); origin xyz=0.0028245 0 0.031696 rpy=0 0 0 -> xyz=0.00032142 0 0.047999 rpy=0 0 0
- joint middle_mcp_roll: axis 1 0 0 -> 0.99996 -0.0086973 0.0018472; limit lower=-0.23 upper=0.23 effort=100 velocity=1 -> lower=-0.267 upper=0.267 effort=0 velocity=0; origin xyz=0.00379999999265848 -0.0117500000029305 0.1526 rpy=0 0 0 -> xyz=-0.0024054 -0.011129 0.10418 rpy=0 0 0
- joint middle_pip: axis 0 1 0 -> 0 1 1.3016E-05; limit lower=0 upper=1.74 effort=100 velocity=1 -> lower=0 upper=1.9548 effort=0 velocity=0; origin xyz=-0.00419457745591796 0 0.0448194332262389 rpy=0 0 0 -> xyz=0.014909 0 0.0135 rpy=0 0 0; parent middle_proximal -> middle_metacarpals
- joint pinky_dip: axis 0 1 0 -> 0 1 1.7355E-05; limit lower=0 upper=1.55 effort=100 velocity=1 -> lower=0 upper=1.9897 effort=0 velocity=0; mimic joint=pinky_pip multiplier=0.89 offset=0 -> (none); origin xyz=0.0028245 0 0.031696 rpy=0 0 0 -> xyz=0.00032142 0 0.047999 rpy=0 0 0
- joint pinky_mcp_roll: axis 1 0 0 -> 0.99996 0.0088916 0; limit lower=-0.23 upper=0.23 effort=100 velocity=1 -> lower=-0.2182 upper=0.08726 effort=0 velocity=0; origin xyz=0.00379999999998499 0.0352499999970695 0.1436 rpy=0 0 0 -> xyz=-0.0024054 0.030888 0.081471 rpy=0 0 0
- joint pinky_pip: axis 0 1 0 -> 0 1 1.3016E-05; limit lower=0 upper=1.74 effort=100 velocity=1 -> lower=0 upper=1.9548 effort=0 velocity=0; origin xyz=-0.0041946 0 0.044819 rpy=0 0 0 -> xyz=0.014909 0 0.0135 rpy=0 0 0; parent pinky_proximal -> pinky_metacarpals
- joint ring_dip: axis 0 1 0 -> 0 1 1.7355E-05; limit lower=0 upper=1.55 effort=100 velocity=1 -> lower=0 upper=1.9897 effort=0 velocity=0; mimic joint=ring_pip multiplier=0.89 offset=0 -> (none); origin xyz=0.0028245 0 0.031696 rpy=0 0 0 -> xyz=0.00032142 0 0.047999 rpy=0 0 0
- joint ring_mcp_roll: axis 1 0 0 -> 0.99996 0.0086973 0.0018472; limit lower=-0.23 upper=0.23 effort=100 velocity=1 -> lower=-0.1920 upper=0.2112 effort=0 velocity=0; origin xyz=0.00379999999632174 0.0117499999970695 0.1481 rpy=0 0 0 -> xyz=-0.0024054 0.009871 0.095682 rpy=0 0 0
- joint ring_pip: axis 0 1 0 -> 0 1 1.3016E-05; limit lower=0 upper=1.74 effort=100 velocity=1 -> lower=0 upper=1.9548 effort=0 velocity=0; origin xyz=-0.00419457745591796 0 0.0448194332262389 rpy=0 0 0 -> xyz=0.014909 0 0.0135 rpy=0 0 0; parent ring_proximal -> ring_metacarpals
- joint thumb_cmc_roll: axis -1 0 0 -> 1 0 0; limit lower=0 upper=1.4 effort=100 velocity=1 -> lower=-0.5236 upper=0.5236 effort=0 velocity=0; origin xyz=0.01916 -0.01 0.0436 rpy=0 0 0 -> xyz=0.0084485 -0.024335 0.042911 rpy=0 0 0
- joint thumb_cmc_yaw: axis 0 0 1 -> 0 0 0.999999999998969; limit lower=0 upper=1.57 effort=100 velocity=1 -> lower=-1.574 upper=0.628 effort=0 velocity=0; origin xyz=0.019845 0 0 rpy=0.77165 0 0 -> xyz=0.0159999999998202 -0.00610000000001085 0 rpy=0 0 0
- joint thumb_mcp: axis 0 1 0 -> 0.0130552606816428 -0.999914776314982 -1.65980330510397E-05; limit lower=0 upper=1.26 effort=100 velocity=1 -> lower=0 upper=1.169 effort=0 velocity=0; origin xyz=0.0127018248047608 0 0.0627256157349894 rpy=0 0 0 -> xyz=0.0169416180142918 0.00322287013353829 0.00617135682158507 rpy=0 0 0; parent thumb_metacarpals -> thumb_metacarpals_base2

File: src/linkerhand_retarget/linkerhand_retarget/assets/robots/hands/linker_hand/o20_right/linkerhand_o20_right.urdf (robot description, URDF)
Before this commit: robot linkerhand_o20_right.urdf, 22 links, 21 joints
Links:
- removed link hand_base_link
- removed link index_distal
- removed link index_metacarpals
- removed link index_middle
- removed link index_proximal
- removed link middle_distal
- removed link middle_metacarpals
- removed link middle_middle
- removed link middle_proximal
- removed link pinky_distal
- removed link pinky_metacarpals
- removed link pinky_middle
- removed link pinky_proximal
- removed link ring_distal
- removed link ring_metacarpals
- removed link ring_middle
- removed link ring_proximal
- removed link thumb_distal
- removed link thumb_metacarpals
- removed link thumb_metacarpals_base1
- removed link thumb_metacarpals_base2
- removed link thumb_proximal
- added link hand_link, mass 0.057077336429848; collision mesh filename=meshes/hand_link.STL; visual mesh filename=meshes/hand_link.STL
- added link index_distal_Link, mass 0.0040079652611257; collision mesh filename=meshes/index_distal_Link.STL; visual mesh filename=meshes/index_distal_Link.STL
- added link index_metacarpals_Link, mass 0.0073508478100444; collision mesh filename=meshes/index_metacarpals_Link.STL; visual mesh filename=meshes/index_metacarpals_Link.STL
- added link index_proximal_Link, mass 0.00831558077334137; collision mesh filename=meshes/index_proximal_Link.STL; visual mesh filename=meshes/index_proximal_Link.STL
- added link middle_distal_Link, mass 0.0040079649798981; collision mesh filename=meshes/middle_distal_Link.STL; visual mesh filename=meshes/middle_distal_Link.STL
- added link middle_metacarpals_Link, mass 0.00735084781003671; collision mesh filename=meshes/middle_metacarpals_Link.STL; visual mesh filename=meshes/middle_metacarpals_Link.STL
- added link middle_proximal_Link, mass 0.00831558078101827; collision mesh filename=meshes/middle_proximal_Link.STL; visual mesh filename=meshes/middle_proximal_Link.STL
- added link pinky_distal_Link, mass 0.00400796649887908; collision mesh filename=meshes/pinky_distal_Link.STL; visual mesh filename=meshes/pinky_distal_Link.STL
- added link pinky_metacarpals_Link, mass 0.00735084795302498; collision mesh filename=meshes/pinky_metacarpals_Link.STL; visual mesh filename=meshes/pinky_metacarpals_Link.STL
- added link pinky_proximal_Link, mass 0.00831558077292084; collision mesh filename=meshes/pinky_proximal_Link.STL; visual mesh filename=meshes/pinky_proximal_Link.STL
- added link ring_distal_Link, mass 0.00400796201164192; collision mesh filename=meshes/ring_distal_Link.STL; visual mesh filename=meshes/ring_distal_Link.STL
- added link ring_metacarpals_Link, mass 0.0073508478100305; collision mesh filename=meshes/ring_metacarpals_Link.STL; visual mesh filename=meshes/ring_metacarpals_Link.STL
- added link ring_proximal_Link, mass 0.00831558078090548; collision mesh filename=meshes/ring_proximal_Link.STL; visual mesh filename=meshes/ring_proximal_Link.STL
- added link thumb_metacarpals_Link, mass 0.00844249886138397; collision mesh filename=meshes/thumb_metacarpals_Link.STL; visual mesh filename=meshes/thumb_metacarpals_Link.STL
- added link thumb_metacarpals_base1_Link, mass 0.00845243302462251; collision mesh filename=meshes/thumb_metacarpals_base1_Link.STL; visual mesh filename=meshes/thumb_metacarpals_base1_Link.STL
- added link thumb_metacarpals_base2_Link, mass 0.00107216679298397; collision mesh filename=meshes/thumb_metacarpals_base2_Link.STL; visual mesh filename=meshes/thumb_metacarpals_base2_Link.STL
- added link thumb_proximal_Link, mass 0.00697217500001587; collision mesh filename=meshes/thumb_proximal_Link.STL; visual mesh filename=meshes/thumb_proximal_Link.STL
Joints:
- removed joint index_pip
- removed joint middle_pip
- removed joint pinky_pip
- removed joint ring_pip
- removed joint thumb_ip
- joint index_dip: child index_distal -> index_distal_Link; limit lower=0 upper=1.55 effort=1 velocity=100 -> lower=0 upper=1.85 effort=1 velocity=1; mimic joint=index_pip multiplier=0.89 offset=0 -> (none); origin xyz=0.0028245 0 0.031696 rpy=0 0 0 -> xyz=0.0003221 0 0.047987 rpy=0 0 0; parent index_middle -> index_proximal_Link
- joint index_mcp_pitch: child index_proximal -> index_proximal_Link; limit lower=0 upper=1.22 effort=1 velocity=100 -> lower=0 upper=1.85 effort=1 velocity=1; origin xyz=-0.0021302 0 0 rpy=0 0 0 -> xyz=-0.00506 0 0.0135 rpy=0 0 0; parent index_metacarpals -> index_metacarpals_Link
- joint index_mcp_roll: child index_metacarpals -> index_metacarpals_Link; limit lower=-0.23 upper=0.23 effort=1 velocity=100 -> lower=-0.35 upper=0.09 effort=1 velocity=1; origin xyz=0.0038 0.03525 0.1481 rpy=0 0 0 -> xyz=0.017464 0.032129 0.092682 rpy=0 0 0; parent hand_base_link -> hand_link
- joint middle_dip: child middle_distal -> middle_distal_Link; limit lower=0 upper=1.55 effort=1 velocity=100 -> lower=0 upper=1.85 effort=1 velocity=1; mimic joint=middle_pip multiplier=0.89 offset=0 -> (none); origin xyz=0.0028245 0 0.031696 rpy=0 0 0 -> xyz=0.0003221 0 0.047987 rpy=0 0 0; parent middle_middle -> middle_proximal_Link
- joint middle_mcp_pitch: child middle_proximal -> middle_proximal_Link; limit lower=0 upper=1.22 effort=1 velocity=100 -> lower=0 upper=1.85 effort=1 velocity=1; origin xyz=-0.0021302 0 0 rpy=0 0 0 -> xyz=-0.00506 0 0.0135 rpy=0 0 0; parent middle_metacarpals -> middle_metacarpals_Link
- joint middle_mcp_roll: axis 1 0 0 -> -1 0 0; child middle_metacarpals -> middle_metacarpals_Link; limit lower=-0.23 upper=0.23 effort=1 velocity=100 -> lower=-0.26 upper=0.26 effort=1 velocity=1; origin xyz=0.0038 0.01175 0.1526 rpy=0 0 0 -> xyz=0.017463 0.011129 0.10118 rpy=0 0 0; parent hand_base_link -> hand_link
- joint pinky_dip: child pinky_distal -> pinky_distal_Link; limit lower=0 upper=1.55 effort=1 velocity=100 -> lower=0 upper=1.85 effort=1 velocity=1; mimic joint=pinky_pip multiplier=0.89 offset=0 -> (none); origin xyz=0.0028245 0 0.031696 rpy=0 0 0 -> xyz=0.0003221 0 0.047987 rpy=0 0 0; parent pinky_middle -> pinky_proximal_Link
- joint pinky_mcp_pitch: child pinky_proximal -> pinky_proximal_Link; limit lower=0 upper=1.22 effort=1 velocity=100 -> lower=0 upper=1.85 effort=1 velocity=1; origin xyz=-0.0021302 0 0 rpy=0 0 0 -> xyz=-0.00506 0 0.0135 rpy=-1.3016E-05 0 0; parent pinky_metacarpals -> pinky_metacarpals_Link
- joint pinky_mcp_roll: axis 1 0 0 -> -1 0 0; child pinky_metacarpals -> pinky_metacarpals_Link; limit lower=-0.23 upper=0.23 effort=1 velocity=100 -> lower=-0.21 upper=0.09 effort=1 velocity=1; origin xyz=0.0038 -0.03525 0.1436 rpy=0 0 0 -> xyz=0.017463 -0.030888 0.078471 rpy=0 0 0; parent hand_base_link -> hand_link
- joint ring_dip: child ring_distal -> ring_distal_Link; limit lower=0 upper=1.55 effort=1 velocity=100 -> lower=0 upper=1.85 effort=1 velocity=1; mimic joint=ring_pip multiplier=0.89 offset=0 -> (none); origin xyz=0.0028245 0 0.031696 rpy=0 0 0 -> xyz=0.0003221 0 0.047987 rpy=0 0 0; parent ring_middle -> ring_proximal_Link
- joint ring_mcp_pitch: child ring_proximal -> ring_proximal_Link; limit lower=0 upper=1.22 effort=1 velocity=100 -> lower=0 upper=1.85 effort=1 velocity=1; origin xyz=-0.0021302 0 0 rpy=0 0 0 -> xyz=-0.00506 0 0.0135 rpy=0 0 0; parent ring_metacarpals -> ring_metacarpals_Link
- joint ring_mcp_roll: axis 1 0 0 -> -1 0 0; child ring_metacarpals -> ring_metacarpals_Link; limit lower=-0.23 upper=0.23 effort=1 velocity=100 -> lower=-0.2 upper=0.2 effort=1 velocity=1; origin xyz=0.0038 -0.01175 0.1481 rpy=0 0 0 -> xyz=0.017463 -0.009871 0.092682 rpy=0 0 0; parent hand_base_link -> hand_link
- joint thumb_cmc_pitch: child thumb_metacarpals -> thumb_metacarpals_Link; limit lower=0 upper=0.83 effort=1 velocity=100 -> lower=0 upper=1.17 effort=1 velocity=1; origin xyz=0.0088264 0.024243 0.0005 rpy=0 -1.0647 -1.9199 -> xyz=0.0060748 0.0031232 0.016968 rpy=-0.013414 0.23743 -0.0031552; parent thumb_metacarpals_base2 -> thumb_metacarpals_base2_Link
- joint thumb_cmc_roll: axis 1 0 0 -> 0 0 1; child thumb_metacarpals_base1 -> thumb_metacarpals_base1_Link; limit lower=0 upper=1.39 effort=1 velocity=100 -> lower=-0.52 upper=0.52 effort=1 velocity=1; origin xyz=0.01916 0.01 0.0436 rpy=0 0 0 -> xyz=-0.00014989 0.024335 0.039911 rpy=-3.1139 -1.5708 -0.027697; parent hand_base_link -> hand_link
- joint thumb_cmc_yaw: axis 0 0 -1 -> 1 0 0; child thumb_metacarpals_base2 -> thumb_metacarpals_base2_Link; limit lower=0 upper=1.57 effort=1 velocity=100 -> lower=-0.63 upper=1.57 effort=1 velocity=1; origin xyz=0.019845 0 0 rpy=-0.77165 0 0 -> xyz=0 -0.006 0.024598 rpy=0 0 0; parent thumb_metacarpals_base1 -> thumb_metacarpals_base1_Link
- joint thumb_mcp: child thumb_proximal -> thumb_proximal_Link; limit lower=0 upper=1.25 effort=1 velocity=100 -> lower=0 upper=1.57 effort=1 velocity=1; origin xyz=0.012702 0 0.062726 rpy=0 0 0 -> xyz=0 0 0.051013 rpy=0 0 0; parent thumb_metacarpals -> thumb_metacarpals_Link

Commit message: 修复多机型标定缓存并补充O30i接入

File: src/linkerhand_retarget/linkerhand_retarget/assets/robots/hands/linker_hand/o20_left/linkerhand_o20_left.urdf (robot description, URDF)
Before this commit: robot linkerhand_O20_lefthand, 17 links, 16 joints
Joints:
- joint thumb_cmc_yaw: limit lower=-1.574 upper=0.628 effort=0 velocity=0 -> lower=-1.574 upper=0 effort=0 velocity=0

File: src/linkerhand_retarget/linkerhand_retarget/assets/robots/hands/linker_hand/o20_right/linkerhand_o20_right.urdf (robot description, URDF)
Before this commit: robot linkerhand_o20_right, 17 links, 16 joints
Joints:
- joint thumb_cmc_yaw: limit lower=-0.63 upper=1.57 effort=1 velocity=1 -> lower=0 upper=1.57 effort=1 velocity=1
