Commit message: refactor: canonicalize customer o30 model

File: src/linkerhand_retarget/linkerhand_retarget/assets/robots/hands/linker_hand/g20_left/linkerhand_g20_left.urdf (robot description, URDF)
Before this commit: robot linkerhand_g20_left.urdf, 22 links, 21 joints
Joints:
- joint index_mcp_pitch: limit lower=0 upper=1.22 effort=100 velocity=1 -> lower=0 upper=1.23297265625997 effort=100 velocity=1
- joint index_mcp_roll: limit lower=-0.23 upper=0.23 effort=100 velocity=1 -> lower=-0.259862986259972 upper=0.256863626259972 effort=100 velocity=1
- joint index_pip: limit lower=0 upper=1.74 effort=100 velocity=1 -> lower=0 upper=1.75088443625997 effort=100 velocity=1
- joint middle_mcp_pitch: limit lower=0 upper=1.22 effort=100 velocity=1 -> lower=0 upper=1.23297265625997 effort=100 velocity=1
- joint middle_mcp_roll: limit lower=-0.23 upper=0.23 effort=100 velocity=1 -> lower=-0.259862986259972 upper=0.256863626259972 effort=100 velocity=1
- joint middle_pip: limit lower=0 upper=1.74 effort=100 velocity=1 -> lower=0 upper=1.75088443625997 effort=100 velocity=1
- joint pinky_mcp_pitch: limit lower=0 upper=1.22 effort=100 velocity=1 -> lower=0 upper=1.23297265625997 effort=100 velocity=1
- joint pinky_mcp_roll: limit lower=-0.23 upper=0.23 effort=100 velocity=1 -> lower=-0.259862986259972 upper=0.256863626259972 effort=100 velocity=1
- joint pinky_pip: limit lower=0 upper=1.74 effort=100 velocity=1 -> lower=0 upper=1.75088443625997 effort=100 velocity=1
- joint ring_mcp_pitch: limit lower=0 upper=1.22 effort=100 velocity=1 -> lower=0 upper=1.23297265625997 effort=100 velocity=1
- joint ring_mcp_roll: limit lower=-0.23 upper=0.23 effort=100 velocity=1 -> lower=-0.259862986259972 upper=0.256863626259972 effort=100 velocity=1
- joint ring_pip: limit lower=0 upper=1.74 effort=100 velocity=1 -> lower=0 upper=1.75088443625997 effort=100 velocity=1
- joint thumb_cmc_pitch: origin xyz=0.0088218 -0.024245 0.0005 rpy=0 -1.0647 1.9199 -> xyz=0.0088218 -0.024245 0.0005 rpy=2.22044604925031e-16 -1.01444006 1.9199
- joint thumb_cmc_roll: origin xyz=0.01916 -0.01 0.0436 rpy=0 0 0 -> xyz=0.01916 -0.01 0.0436 rpy=-0.122173047639603 0 0
- joint thumb_cmc_yaw: origin xyz=0.019845 0 0 rpy=0.77165 0 0 -> xyz=0.019845 0 0 rpy=0.771494635674502 0.017384990508633 -0.0178724603975689

File: src/linkerhand_retarget/linkerhand_retarget/assets/robots/hands/linker_hand/g20_right/linkerhand_g20_right.urdf (robot description, URDF)
Before this commit: robot linkerhand_L25NS_right.urdf, 22 links, 21 joints
Joints:
- joint thumb_cmc_pitch: origin xyz=0.0088264 0.024243 0.0005 rpy=0 -1.0647 -1.9199 -> xyz=0.0088264 0.024243 0.0005 rpy=-4.44089209850063e-16 -1.03160184765982 -1.9199
- joint thumb_cmc_roll: origin xyz=0.01916 0.01 0.0436 rpy=0 0 0 -> xyz=0.01916 0.01 0.0436 rpy=0.0669047936042155 0 0
- joint thumb_cmc_yaw: origin xyz=0.019845 0 0 rpy=-0.77165 0 0 -> xyz=0.019845 0 0 rpy=-0.771519235634338 -0.015949629057757 -0.0163964520694657

File: src/linkerhand_retarget/linkerhand_retarget/assets/robots/hands/linker_hand/o30_left/linkerhand_o30_left.urdf (robot description, URDF)
Before this commit: robot linkerhand_o30_left.urdf, 22 links, 21 joints
Links:
- removed link thumb_metacarpals
- link hand_base_link: mass 0.110373495507463 -> 0.0570701007302751; geometry collision mesh filename=meshes/hand_base_link.STL scale=1.0 -1.0 1.0; visual mesh filename=meshes/hand_base_link.STL scale=1.0 -1.0 1.0
- link index_distal: mass 0.00334170259772608 -> 0.0033098791304967; geometry collision mesh filename=meshes/index_distal.STL scale=1.0 -1.0 1.0; visual mesh filename=meshes/index_distal.STL scale=1.0 -1.0 1.0
- link index_metacarpals: mass 0.000895516429792169 -> 0.00661261244742178; geometry collision mesh filename=meshes/index_metacarpals.STL scale=1.0 -1.0 1.0; visual mesh filename=meshes/index_metacarpals.STL scale=1.0 -1.0 1.0
- link index_middle: mass 0.00237827499847615 -> 0.00678023137976301; geometry collision mesh filename=meshes/index_middle.STL scale=1.0 -1.0 1.0; visual mesh filename=meshes/index_middle.STL scale=1.0 -1.0 1.0
- link index_proximal: mass 0.00450921353606138 -> 0.00727256326100808; geometry collision mesh filename=meshes/index_proximal.STL scale=1.0 -1.0 1.0; visual mesh filename=meshes/index_proximal.STL scale=1.0 -1.0 1.0
- link middle_distal: mass 0.00334170288968694 -> 0.00330988759550385; geometry collision mesh filename=meshes/middle_distal.STL scale=1.0 -1.0 1.0; visual mesh filename=meshes/middle_distal.STL scale=1.0 -1.0 1.0
- link middle_metacarpals: mass 0.000895516947435045 -> 0.00661261244742176; geometry collision mesh filename=meshes/middle_metacarpals.STL scale=1.0 -1.0 1.0; visual mesh filename=meshes/middle_metacarpals.STL scale=1.0 -1.0 1.0
- link middle_middle: mass 0.00237827502274046 -> 0.00558395826725584; geometry collision mesh filename=meshes/middle_middle.STL scale=1.0 -1.0 1.0; visual mesh filename=meshes/middle_middle.STL scale=1.0 -1.0 1.0
- link middle_proximal: mass 0.00450921353536659 -> 0.00727256322379252; geometry collision mesh filename=meshes/middle_proximal.STL scale=1.0 -1.0 1.0; visual mesh filename=meshes/middle_proximal.STL scale=1.0 -1.0 1.0
- link pinky_distal: mass 0.00334170283969146 -> 0.00330987874289192; geometry collision mesh filename=meshes/pinky_distal.STL scale=1.0 -1.0 1.0; visual mesh filename=meshes/pinky_distal.STL scale=1.0 -1.0 1.0
- link pinky_metacarpals: mass 0.000895516947513541 -> 0.00661261244414956; geometry collision mesh filename=meshes/pinky_metacarpals.STL scale=1.0 -1.0 1.0; visual mesh filename=meshes/pinky_metacarpals.STL scale=1.0 -1.0 1.0
- link pinky_middle: mass 0.00237827431921004 -> 0.00678023141445045; geometry collision mesh filename=meshes/pinky_middle.STL scale=1.0 -1.0 1.0; visual mesh filename=meshes/pinky_middle.STL scale=1.0 -1.0 1.0
- link pinky_proximal: mass 0.00450921353949741 -> 0.00727256322451616; geometry collision mesh filename=meshes/pinky_proximal.STL scale=1.0 -1.0 1.0; visual mesh filename=meshes/pinky_proximal.STL scale=1.0 -1.0 1.0
- link ring_distal: mass 0.00334170280386792 -> 0.00330988375961977; geometry collision mesh filename=meshes/ring_distal.STL scale=1.0 -1.0 1.0; visual mesh filename=meshes/ring_distal.STL scale=1.0 -1.0 1.0
- link ring_metacarpals: mass 0.000895516612684195 -> 0.00661261244414956; geometry collision mesh filename=meshes/ring_metacarpals.STL scale=1.0 -1.0 1.0; visual mesh filename=meshes/ring_metacarpals.STL scale=1.0 -1.0 1.0
- link ring_middle: mass 0.00237827433282015 -> 0.00558395830757745; geometry collision mesh filename=meshes/ring_middle.STL scale=1.0 -1.0 1.0; visual mesh filename=meshes/ring_middle.STL scale=1.0 -1.0 1.0
- link ring_proximal: mass 0.00450921353946778 -> 0.00727256326396366; geometry collision mesh filename=meshes/ring_proximal.STL scale=1.0 -1.0 1.0; visual mesh filename=meshes/ring_proximal.STL scale=1.0 -1.0 1.0
- link thumb_distal: mass 0.00382046638843239 -> 0.0033703198194942; geometry collision mesh filename=meshes/thumb_distal.STL scale=1.0 -1.0 1.0; visual mesh filename=meshes/thumb_distal.STL scale=1.0 -1.0 1.0
- link thumb_metacarpals_base1: mass 0.0160351802817401 -> 0.00628309017011841; geometry collision mesh filename=meshes/thumb_metacarpals_base1.STL scale=1.0 -1.0 1.0; visual mesh filename=meshes/thumb_metacarpals_base1.STL scale=1.0 -1.0 1.0
- link thumb_metacarpals_base2: mass 0.00183264554882498 -> 0.0124355946309777; geometry collision mesh filename=meshes/thumb_metacarpals_base2.STL scale=1.0 -1.0 1.0; visual mesh filename=meshes/thumb_metacarpals_base2.STL scale=1.0 -1.0 1.0
- link thumb_proximal: mass 0.00549015507433734 -> 0.00973720424636687; geometry collision mesh filename=meshes/thumb_proximal.STL scale=1.0 -1.0 1.0; visual mesh filename=meshes/thumb_proximal.STL scale=1.0 -1.0 1.0
Joints:
- removed joint thumb_cmc_pitch
- removed joint thumb_ip
- added joint thumb_dip: type revolute, parent thumb_proximal, child thumb_distal, origin xyz=4.8488e-05 -0.040032 -0.0005 rpy=0.0 -0.0 -0.0, axis -1.0 0.0 0.0, limit lower=0.0 upper=1.66 effort=1.0 velocity=1.0
- joint index_dip: axis 0 1 0 -> 0.0 1.0 0.0; limit lower=0 upper=1.55 effort=100 velocity=1 -> lower=0 upper=1.55 effort=1.0 velocity=1.0; mimic joint=index_pip multiplier=0.89 offset=0 -> (none); origin xyz=0.0028245 0 0.031696 rpy=0 0 0 -> xyz=0.0 -0.0 0.040244 rpy=0.0 0.0 -0.0
- joint index_mcp_pitch: axis 0 1 0 -> 0.0 1.0 0.0; limit lower=0 upper=1.22 effort=100 velocity=1 -> lower=0.0 upper=1.77 effort=1.0 velocity=1.0; origin xyz=-0.0021302 0 0 rpy=0 0 0 -> xyz=-0.00475 -0.00059587 0.016238 rpy=0.0 0.0 -0.0
- joint index_mcp_roll: axis 1 0 0 -> 1.0 0.0 0.0; limit lower=-0.23 upper=0.23 effort=100 velocity=1 -> lower=-0.07 upper=0.4 effort=1.0 velocity=1.0; origin xyz=0.0038 -0.03525 0.1481 rpy=0 0 0 -> xyz=0.018722 -0.029679 0.075158 rpy=0.0 0.0 -0.0
- joint index_pip: axis 0 1 0 -> 0.0 1.0 0.0; limit lower=0 upper=1.74 effort=100 velocity=1 -> lower=0.0 upper=1.63 effort=1.0 velocity=1.0; origin xyz=-0.0041946 0 0.044819 rpy=0 0 0 -> xyz=0.0 -0.0 0.039681 rpy=0.0 0.0 -0.0
- joint middle_dip: axis 0 1 0 -> 0.0 1.0 0.0; limit lower=0 upper=1.55 effort=100 velocity=1 -> lower=0.0 upper=1.55 effort=1.0 velocity=1.0; mimic joint=middle_pip multiplier=0.89 offset=0 -> (none); origin xyz=0.0028245 0 0.031696 rpy=0 0 0 -> xyz=0.0 -0.0 0.040244 rpy=0.0 0.0 -0.0
- joint middle_mcp_pitch: axis 0 1 0 -> 0.0 1.0 0.0; limit lower=0 upper=1.22 effort=100 velocity=1 -> lower=0.0 upper=1.77 effort=1.0 velocity=1.0; origin xyz=-0.0021302 0 0 rpy=0 0 0 -> xyz=-0.00475 -0.00059587 0.016238 rpy=0.0 0.0 -0.0
- joint middle_mcp_roll: axis 1 0 0 -> 1.0 0.0 0.0; limit lower=-0.23 upper=0.23 effort=100 velocity=1 -> lower=-0.26 upper=0.38 effort=1.0 velocity=1.0; origin xyz=0.00379999999265848 -0.0117500000029305 0.1526 rpy=0 0 0 -> xyz=0.018722 -0.0086937 0.081586 rpy=0.0 0.0 -0.0
- joint middle_pip: axis 0 1 0 -> 0.0 1.0 0.0; limit lower=0 upper=1.74 effort=100 velocity=1 -> lower=0.0 upper=1.63 effort=1.0 velocity=1.0; origin xyz=-0.00419457745591796 0 0.0448194332262389 rpy=0 0 0 -> xyz=0.0 -0.0 0.039681 rpy=0.0 0.0 -0.0
- joint pinky_dip: axis 0 1 0 -> 0.0 1.0 0.0; limit lower=0 upper=1.55 effort=100 velocity=1 -> lower=0.0 upper=1.55 effort=1.0 velocity=1.0; mimic joint=pinky_pip multiplier=0.89 offset=0 -> (none); origin xyz=0.0028245 0 0.031696 rpy=0 0 0 -> xyz=0.0 -0.0 0.040244 rpy=0.0 0.0 -0.0
- joint pinky_mcp_pitch: axis 0 1 0 -> 0.0 1.0 0.0; limit lower=0 upper=1.22 effort=100 velocity=1 -> lower=0.0 upper=1.77 effort=1.0 velocity=1.0; origin xyz=-0.0021302 0 0 rpy=0 0 0 -> xyz=-0.00475 -0.00059587 0.016238 rpy=0.0 0.0 -0.0
- joint pinky_mcp_roll: axis 1 0 0 -> 1.0 0.0 0.0; limit lower=-0.23 upper=0.23 effort=100 velocity=1 -> lower=-0.17 upper=0.28 effort=1.0 velocity=1.0; origin xyz=0.00379999999998499 0.0352499999970695 0.1436 rpy=0 0 0 -> xyz=0.018722 0.030927 0.067761 rpy=0.0 0.0 -0.0
- joint pinky_pip: axis 0 1 0 -> 0.0 1.0 0.0; limit lower=0 upper=1.74 effort=100 velocity=1 -> lower=0.0 upper=1.63 effort=1.0 velocity=1.0; origin xyz=-0.0041946 0 0.044819 rpy=0 0 0 -> xyz=0.0 -0.0 0.039681 rpy=0.0 0.0 -0.0
- joint ring_dip: axis 0 1 0 -> 0.0 1.0 0.0; limit lower=0 upper=1.55 effort=100 velocity=1 -> lower=0.0 upper=1.55 effort=1.0 velocity=1.0; mimic joint=ring_pip multiplier=0.89 offset=0 -> (none); origin xyz=0.0028245 0 0.031696 rpy=0 0 0 -> xyz=0.0 -0.0 0.040244 rpy=0.0 0.0 -0.0
- joint ring_mcp_pitch: axis 0 1 0 -> 0.0 1.0 0.0; limit lower=0 upper=1.22 effort=100 velocity=1 -> lower=0.0 upper=1.77 effort=1.0 velocity=1.0; origin xyz=-0.0021302 0 0 rpy=0 0 0 -> xyz=-0.00475 -0.00059587 0.016238 rpy=0.0 0.0 -0.0
- joint ring_mcp_roll: axis 1 0 0 -> 1.0 0.0 0.0; limit lower=-0.23 upper=0.23 effort=100 velocity=1 -> lower=-0.17 upper=0.28 effort=0.0 velocity=0.0; origin xyz=0.00379999999632174 0.0117499999970695 0.1481 rpy=0 0 0 -> xyz=0.018722 0.012188 0.079218 rpy=0.0 0.0 -0.0
- joint ring_pip: axis 0 1 0 -> 0.0 1.0 0.0; limit lower=0 upper=1.74 effort=100 velocity=1 -> lower=0.0 upper=1.63 effort=1.0 velocity=1.0; origin xyz=-0.00419457745591796 0 0.0448194332262389 rpy=0 0 0 -> xyz=0.0 -0.0 0.039681 rpy=0.0 0.0 -0.0
- joint thumb_cmc_roll: axis -1 0 0 -> -1.0 0.0 0.0; limit lower=0 upper=1.4 effort=100 velocity=1 -> lower=0.0 upper=0.6108 effort=1.0 velocity=1.0; origin xyz=0.01916 -0.01 0.0436 rpy=0 0 0 -> xyz=0.018722 -0.016674 0.024272 rpy=0.0 -0.0 -0.0
- joint thumb_cmc_yaw: axis 0 0 1 -> 0.0 0.0 1.0; limit lower=0 upper=1.57 effort=100 velocity=1 -> lower=0.0 upper=1.63 effort=1.0 velocity=1.0; origin xyz=0.019845 0 0 rpy=0.77165 0 0 -> xyz=-0.00475 -0.016238 -0.00059587 rpy=-0.0 0.0 0.0
- joint thumb_mcp: axis 0 1 0 -> -1.0 0.0 0.0; limit lower=0 upper=1.26 effort=100 velocity=1 -> lower=0.0 upper=1.51 effort=1.0 velocity=1.0; origin xyz=0.0127018248047608 0 0.0627256157349894 rpy=0 0 0 -> xyz=-5.4077e-05 -0.052039 0.0059395 rpy=0.0 -0.0 -0.0; parent thumb_metacarpals -> thumb_metacarpals_base2

File: src/linkerhand_retarget/linkerhand_retarget/assets/robots/hands/linker_hand/o30_right/linkerhand_o30_right.urdf (robot description, URDF)
Before this commit: robot linkerhand_o30_right.urdf, 22 links, 21 joints
Links:
- removed link thumb_metacarpals
- link hand_base_link: mass 0.130043890829375 -> 0.0570701007302751
- link index_distal: mass 0.00334176238570705 -> 0.0033098791304967
- link index_metacarpals: mass 0.000895533942236676 -> 0.00661261244742178
- link index_middle: mass 0.00237861824163327 -> 0.00678023137976301
- link index_proximal: mass 0.00450935628154297 -> 0.00727256326100808
- link middle_distal: mass 0.0033417623857295 -> 0.00330988759550385
- link middle_metacarpals: mass 0.000895533942236672 -> 0.00661261244742176
- link middle_middle: mass 0.00237861824399121 -> 0.00558395826725584
- link middle_proximal: mass 0.00450935628154299 -> 0.00727256322379252
- link pinky_distal: mass 0.00334176233214274 -> 0.00330987874289192
- link pinky_metacarpals: mass 0.000895533942236661 -> 0.00661261244414956
- link pinky_middle: mass 0.0023786182416333 -> 0.00678023141445045
- link pinky_proximal: mass 0.00450935627773312 -> 0.00727256322451616
- link ring_distal: mass 0.00334176238553782 -> 0.00330988375961977
- link ring_metacarpals: mass 0.00089553394223667 -> 0.00661261244414956
- link ring_middle: mass 0.00237861824163314 -> 0.00558395830757745
- link ring_proximal: mass 0.00450935628154299 -> 0.00727256326396366
- link thumb_distal: mass 0.00585464206993151 -> 0.0033703198194942
- link thumb_metacarpals_base1: mass 0.0173128324517923 -> 0.00628309017011841
- link thumb_metacarpals_base2: mass 0.0129293097380942 -> 0.0124355946309777
- link thumb_proximal: mass 0.00549015851204037 -> 0.00973720424636687
Joints:
- removed joint thumb_cmc_pitch
- removed joint thumb_ip
- added joint thumb_dip: type revolute, parent thumb_proximal, child thumb_distal, origin xyz=4.8488E-05 0.040032 -0.0005 rpy=0 0 0, axis 1 0 0, limit lower=0 upper=1.66 effort=1 velocity=1
- joint index_dip: limit lower=0 upper=1.55 effort=1 velocity=100 -> lower=0 upper=1.55 effort=1 velocity=1; mimic joint=index_pip multiplier=0.89 offset=0 -> (none); origin xyz=0.0028245 0 0.031696 rpy=0 0 0 -> xyz=0 0 0.040244 rpy=0 0 0
- joint index_mcp_pitch: limit lower=0 upper=1.22 effort=1 velocity=100 -> lower=0 upper=1.77 effort=1 velocity=1; origin xyz=-0.0021302 0 0 rpy=0 0 0 -> xyz=-0.00475 0.00059587 0.016238 rpy=0 0 0
- joint index_mcp_roll: axis 1 0 0 -> -1 0 0; limit lower=-0.23 upper=0.23 effort=1 velocity=100 -> lower=-0.07 upper=0.4 effort=1 velocity=1; origin xyz=0.0038 0.03525 0.1481 rpy=0 0 0 -> xyz=0.018722 0.029679 0.075158 rpy=0 0 0
- joint index_pip: limit lower=0 upper=1.75 effort=1 velocity=100 -> lower=0 upper=1.63 effort=1 velocity=1; origin xyz=-0.0041946 0 0.044819 rpy=0 0 0 -> xyz=0 0 0.039681 rpy=0 0 0
- joint middle_dip: limit lower=0 upper=1.55 effort=1 velocity=100 -> lower=0 upper=1.55 effort=1 velocity=1; mimic joint=middle_pip multiplier=0.89 offset=0 -> (none); origin xyz=0.0028245 0 0.031696 rpy=0 0 0 -> xyz=0 0 0.040244 rpy=0 0 0
- joint middle_mcp_pitch: limit lower=0 upper=1.22 effort=1 velocity=100 -> lower=0 upper=1.77 effort=1 velocity=1; origin xyz=-0.0021302 0 0 rpy=0 0 0 -> xyz=-0.00475 0.00059587 0.016238 rpy=0 0 0
- joint middle_mcp_roll: axis 1 0 0 -> -1 0 0; limit lower=-0.23 upper=0.23 effort=1 velocity=100 -> lower=-0.26 upper=0.38 effort=1 velocity=1; origin xyz=0.0038 0.01175 0.1526 rpy=0 0 0 -> xyz=0.018722 0.0086937 0.081586 rpy=0 0 0
- joint middle_pip: limit lower=0 upper=1.75 effort=1 velocity=100 -> lower=0 upper=1.63 effort=1 velocity=1; origin xyz=-0.0041946 0 0.044819 rpy=0 0 0 -> xyz=0 0 0.039681 rpy=0 0 0
- joint pinky_dip: limit lower=0 upper=1.55 effort=1 velocity=100 -> lower=0 upper=1.55 effort=1 velocity=1; mimic joint=pinky_pip multiplier=0.89 offset=0 -> (none); origin xyz=0.0028245 0 0.031696 rpy=0 0 0 -> xyz=0 0 0.040244 rpy=0 0 0
- joint pinky_mcp_pitch: limit lower=0 upper=1.22 effort=1 velocity=100 -> lower=0 upper=1.77 effort=1 velocity=1; origin xyz=-0.0021302 0 0 rpy=0 0 0 -> xyz=-0.00475 0.00059587 0.016238 rpy=0 0 0
- joint pinky_mcp_roll: axis 1 0 0 -> -1 0 0; limit lower=-0.23 upper=0.23 effort=1 velocity=100 -> lower=-0.17 upper=0.28 effort=1 velocity=1; origin xyz=0.0038 -0.03525 0.1436 rpy=0 0 0 -> xyz=0.018722 -0.030927 0.067761 rpy=0 0 0
- joint pinky_pip: limit lower=0 upper=1.75 effort=1 velocity=100 -> lower=0 upper=1.63 effort=1 velocity=1; origin xyz=-0.0041946 0 0.044819 rpy=0 0 0 -> xyz=0 0 0.039681 rpy=0 0 0
- joint ring_dip: limit lower=0 upper=1.55 effort=1 velocity=100 -> lower=0 upper=1.55 effort=1 velocity=1; mimic joint=ring_pip multiplier=0.89 offset=0 -> (none); origin xyz=0.0028245 0 0.031696 rpy=0 0 0 -> xyz=0 0 0.040244 rpy=0 0 0
- joint ring_mcp_pitch: limit lower=0 upper=1.22 effort=1 velocity=100 -> lower=0 upper=1.77 effort=1 velocity=1; origin xyz=-0.0021302 0 0 rpy=0 0 0 -> xyz=-0.00475 0.00059587 0.016238 rpy=0 0 0
- joint ring_mcp_roll: axis 1 0 0 -> -1 0 0; limit lower=-0.23 upper=0.23 effort=1 velocity=100 -> lower=-0.17 upper=0.28 effort=0 velocity=0; origin xyz=0.0038 -0.01175 0.1481 rpy=0 0 0 -> xyz=0.018722 -0.012188 0.079218 rpy=0 0 0
- joint ring_pip: limit lower=0 upper=1.75 effort=1 velocity=100 -> lower=0 upper=1.63 effort=1 velocity=1; origin xyz=-0.0041946 0 0.044819 rpy=0 0 0 -> xyz=0 0 0.039681 rpy=0 0 0
- joint thumb_cmc_roll: limit lower=0 upper=1.39 effort=1 velocity=100 -> lower=0 upper=0.6108 effort=1 velocity=1; origin xyz=0.01916 0.01 0.0436 rpy=0 0 0 -> xyz=0.018722 0.016674 0.024272 rpy=0 0 0
- joint thumb_cmc_yaw: limit lower=0 upper=1.57 effort=1 velocity=100 -> lower=0 upper=1.63 effort=1 velocity=1; origin xyz=0.019845 0 0 rpy=-0.77165 0 0 -> xyz=-0.00475 0.016238 -0.00059587 rpy=0 0 0
- joint thumb_mcp: axis 0 1 0 -> 1 0 0; limit lower=0 upper=1.25 effort=1 velocity=100 -> lower=0 upper=1.51 effort=1 velocity=1; origin xyz=0.012702 0 0.062726 rpy=0 0 0 -> xyz=-5.4077E-05 0.052039 0.0059395 rpy=0 0 0; parent thumb_metacarpals -> thumb_metacarpals_base2
