Commit message: feat: update O30 model and LinkerForce feedback config

File: src/linkerhand_retarget/linkerhand_retarget/assets/robots/hands/linker_hand/o30_left/linkerhand_o30_left.urdf (robot description, URDF)
Before this commit: robot linkerhand_O30_left.urdf, 21 links, 20 joints
Links:
- link hand_base_link: mass 0.0570701007302751 -> 0.046494
- link thumb_distal: mass 0.0033703198194942 -> 0.0079712
- link thumb_metacarpals_base1: mass 0.00628309017011841 -> 0.0024826
- link thumb_metacarpals_base2: mass 0.0124355946309777 -> 0.0011821
- link thumb_proximal: mass 0.00973720424636687 -> 0.0073969
Joints:
- removed joint thumb_dip
- added joint thumb_ip: type revolute, parent thumb_proximal, child thumb_distal, origin xyz=0.0 -0.048532 0.00155 rpy=-0.0 -0.0 -0.0, axis -1.0 -0.0 -0.0, limit lower=0.0 upper=1.5912 effort=1.0 velocity=1.0
- joint index_dip: limit lower=0 upper=1.55 effort=1.0 velocity=1.0 -> lower=0.0 upper=1.5967 effort=1.0 velocity=1.0; origin xyz=0.0 -0.0 0.040244 rpy=0.0 0.0 -0.0 -> xyz=0.0 -0.0 0.040244 rpy=-0.0 -0.0 -0.0
- joint index_mcp_pitch: limit lower=0.0 upper=1.77 effort=1.0 velocity=1.0 -> lower=0.0 upper=1.8381 effort=1.0 velocity=1.0; origin xyz=-0.00475 -0.00059587 0.016238 rpy=0.0 0.0 -0.0 -> xyz=-0.00475 -0.00059587 0.016238 rpy=-0.0 -0.0 -0.0
- joint index_mcp_roll: axis 1.0 0.0 0.0 -> -1.0 -0.0 -0.0; limit lower=-0.07 upper=0.4 effort=1.0 velocity=1.0 -> lower=-0.397 upper=0.0203 effort=1.0 velocity=1.0; origin xyz=0.018722 -0.029679 0.075158 rpy=0.0 0.0 -0.0 -> xyz=0.018722 -0.029679 0.075158 rpy=-0.0 -0.0 -0.0
- joint index_pip: limit lower=0.0 upper=1.63 effort=1.0 velocity=1.0 -> lower=0.0 upper=1.5958 effort=1.0 velocity=1.0; origin xyz=0.0 -0.0 0.039681 rpy=0.0 0.0 -0.0 -> xyz=0.0 -0.0 0.039681 rpy=-0.0 -0.0 -0.0
- joint middle_dip: limit lower=0.0 upper=1.55 effort=1.0 velocity=1.0 -> lower=0.0 upper=1.5851 effort=1.0 velocity=1.0; origin xyz=0.0 -0.0 0.040244 rpy=0.0 0.0 -0.0 -> xyz=0.0 -0.0 0.040244 rpy=-0.0 -0.0 -0.0
- joint middle_mcp_pitch: limit lower=0.0 upper=1.77 effort=1.0 velocity=1.0 -> lower=0.0 upper=1.8159 effort=1.0 velocity=1.0; origin xyz=-0.00475 -0.00059587 0.016238 rpy=0.0 0.0 -0.0 -> xyz=-0.00475 -0.00059587 0.016238 rpy=-0.0 -0.0 -0.0
- joint middle_mcp_roll: axis 1.0 0.0 0.0 -> -1.0 -0.0 -0.0; limit lower=-0.26 upper=0.38 effort=1.0 velocity=1.0 -> lower=-0.4265 upper=0.1521 effort=1.0 velocity=1.0; origin xyz=0.018722 -0.0086937 0.081586 rpy=0.0 0.0 -0.0 -> xyz=0.018722 -0.0086937 0.081586 rpy=-0.0 -0.0 -0.0
- joint middle_pip: limit lower=0.0 upper=1.63 effort=1.0 velocity=1.0 -> lower=0.0 upper=1.5658 effort=1.0 velocity=1.0; origin xyz=0.0 -0.0 0.039681 rpy=0.0 0.0 -0.0 -> xyz=0.0 -0.0 0.039681 rpy=-0.0 -0.0 -0.0
- joint pinky_dip: limit lower=0.0 upper=1.55 effort=1.0 velocity=1.0 -> lower=0.0 upper=1.5897 effort=1.0 velocity=1.0; origin xyz=0.0 -0.0 0.040244 rpy=0.0 0.0 -0.0 -> xyz=0.0 -0.0 0.040244 rpy=-0.0 -0.0 -0.0
- joint pinky_mcp_pitch: limit lower=0.0 upper=1.77 effort=1.0 velocity=1.0 -> lower=0.0 upper=1.8241 effort=1.0 velocity=1.0; origin xyz=-0.00475 -0.00059587 0.016238 rpy=0.0 0.0 -0.0 -> xyz=-0.00475 -0.00059587 0.016238 rpy=-0.0 -0.0 -0.0
- joint pinky_mcp_roll: axis 1.0 0.0 0.0 -> -1.0 -0.0 -0.0; limit lower=-0.17 upper=0.28 effort=1.0 velocity=1.0 -> lower=-0.0548 upper=0.3874 effort=1.0 velocity=1.0; origin xyz=0.018722 0.030927 0.067761 rpy=0.0 0.0 -0.0 -> xyz=0.018722 0.030927 0.067761 rpy=-0.0 -0.0 -0.0
- joint pinky_pip: limit lower=0.0 upper=1.63 effort=1.0 velocity=1.0 -> lower=0.0 upper=1.5123 effort=1.0 velocity=1.0; origin xyz=0.0 -0.0 0.039681 rpy=0.0 0.0 -0.0 -> xyz=0.0 -0.0 0.039681 rpy=-0.0 -0.0 -0.0
- joint ring_dip: limit lower=0.0 upper=1.55 effort=1.0 velocity=1.0 -> lower=0.0 upper=1.5391 effort=1.0 velocity=1.0; origin xyz=0.0 -0.0 0.040244 rpy=0.0 0.0 -0.0 -> xyz=0.0 -0.0 0.040244 rpy=-0.0 -0.0 -0.0
- joint ring_mcp_pitch: limit lower=0.0 upper=1.77 effort=1.0 velocity=1.0 -> lower=0.0 upper=1.8145 effort=1.0 velocity=1.0; origin xyz=-0.00475 -0.00059587 0.016238 rpy=0.0 0.0 -0.0 -> xyz=-0.00475 -0.00059587 0.016238 rpy=-0.0 -0.0 -0.0
- joint ring_mcp_roll: axis 1.0 0.0 0.0 -> -1.0 -0.0 -0.0; limit lower=-0.17 upper=0.28 effort=0.0 velocity=0.0 -> lower=-0.2288 upper=0.3049 effort=0.0 velocity=0.0; origin xyz=0.018722 0.012188 0.079218 rpy=0.0 0.0 -0.0 -> xyz=0.018722 0.012188 0.079218 rpy=-0.0 -0.0 -0.0
- joint ring_pip: limit lower=0.0 upper=1.63 effort=1.0 velocity=1.0 -> lower=0.0 upper=1.4911 effort=1.0 velocity=1.0; origin xyz=0.0 -0.0 0.039681 rpy=0.0 0.0 -0.0 -> xyz=0.0 -0.0 0.039681 rpy=-0.0 -0.0 -0.0
- joint thumb_cmc_roll: axis -1.0 0.0 0.0 -> -1.0 -0.0 -0.0; limit lower=0.0 upper=0.6108 effort=1.0 velocity=1.0 -> lower=0.0 upper=0.6311 effort=1.0 velocity=1.0; origin xyz=0.018722 -0.016674 0.024272 rpy=0.0 -0.0 -0.0 -> xyz=0.018257 -0.012998 0.024272 rpy=-0.0 -0.0 -0.0
- joint thumb_cmc_yaw: axis 0.0 0.0 1.0 -> -0.0 -0.0 1.0; limit lower=0.0 upper=1.63 effort=1.0 velocity=1.0 -> lower=0.0 upper=1.8718 effort=1.0 velocity=1.0; origin xyz=-0.00475 -0.016238 -0.00059587 rpy=-0.0 0.0 0.0 -> xyz=-0.00215 -0.015238 0.0 rpy=-0.0 -0.0 -0.0
- joint thumb_mcp: axis -1.0 0.0 0.0 -> -1.0 -0.0 -0.0; limit lower=0.0 upper=1.51 effort=1.0 velocity=1.0 -> lower=0.0 upper=1.8337 effort=1.0 velocity=1.0; origin xyz=-5.4077e-05 -0.052039 0.0059395 rpy=0.0 -0.0 -0.0 -> xyz=0.00045 -0.015539 0.0029937 rpy=0.33161 -0.0 -0.0

File: src/linkerhand_retarget/linkerhand_retarget/assets/robots/hands/linker_hand/o30_right/linkerhand_o30_right.urdf (robot description, URDF)
Before this commit: robot linkerhand_O30_right.urdf, 21 links, 20 joints
Links:
- link hand_base_link: mass 0.0570701007302751 -> 0.046494
- link thumb_distal: mass 0.0033703198194942 -> 0.0079712
- link thumb_metacarpals_base1: mass 0.00628309017011841 -> 0.0024826
- link thumb_metacarpals_base2: mass 0.0124355946309777 -> 0.0011821
- link thumb_proximal: mass 0.00973720424636687 -> 0.0073969
Joints:
- removed joint thumb_dip
- added joint thumb_ip: type revolute, parent thumb_proximal, child thumb_distal, origin xyz=0 0.048532 0.00155 rpy=0 0 0, axis 1 0 0, limit lower=0 upper=1.5912 effort=1 velocity=1
- joint index_dip: limit lower=0 upper=1.55 effort=1 velocity=1 -> lower=0.0 upper=1.5967 effort=1.0 velocity=1.0
- joint index_mcp_pitch: limit lower=0 upper=1.77 effort=1 velocity=1 -> lower=0.0 upper=1.8381 effort=1.0 velocity=1.0
- joint index_mcp_roll: axis -1 0 0 -> 1 0 0; limit lower=-0.07 upper=0.4 effort=1 velocity=1 -> lower=-0.3970 upper=0.0203 effort=1.0 velocity=1.0
- joint index_pip: limit lower=0 upper=1.63 effort=1 velocity=1 -> lower=0.0 upper=1.5958 effort=1.0 velocity=1.0
- joint middle_dip: limit lower=0 upper=1.55 effort=1 velocity=1 -> lower=0.0 upper=1.5851 effort=1.0 velocity=1.0
- joint middle_mcp_pitch: limit lower=0 upper=1.77 effort=1 velocity=1 -> lower=0.0 upper=1.8159 effort=1.0 velocity=1.0
- joint middle_mcp_roll: axis -1 0 0 -> 1 0 0; limit lower=-0.26 upper=0.38 effort=1 velocity=1 -> lower=-0.4265 upper=0.1521 effort=1.0 velocity=1.0
- joint middle_pip: limit lower=0 upper=1.63 effort=1 velocity=1 -> lower=0.0 upper=1.5658 effort=1.0 velocity=1.0
- joint pinky_dip: limit lower=0 upper=1.55 effort=1 velocity=1 -> lower=0.0 upper=1.5897 effort=1.0 velocity=1.0
- joint pinky_mcp_pitch: limit lower=0 upper=1.77 effort=1 velocity=1 -> lower=0.0 upper=1.8241 effort=1.0 velocity=1.0
- joint pinky_mcp_roll: axis -1 0 0 -> 1 0 0; limit lower=-0.17 upper=0.28 effort=1 velocity=1 -> lower=-0.0548 upper=0.3874 effort=1.0 velocity=1.0
- joint pinky_pip: limit lower=0 upper=1.63 effort=1 velocity=1 -> lower=0.0 upper=1.5123 effort=1.0 velocity=1.0
- joint ring_dip: limit lower=0 upper=1.55 effort=1 velocity=1 -> lower=0.0 upper=1.5391 effort=1.0 velocity=1.0
- joint ring_mcp_pitch: limit lower=0 upper=1.77 effort=1 velocity=1 -> lower=0.0 upper=1.8145 effort=1.0 velocity=1.0
- joint ring_mcp_roll: axis -1 0 0 -> 1 0 0; limit lower=-0.17 upper=0.28 effort=0 velocity=0 -> lower=-0.2288 upper=0.3049 effort=0.0 velocity=0.0
- joint ring_pip: limit lower=0 upper=1.63 effort=1 velocity=1 -> lower=0.0 upper=1.4911 effort=1.0 velocity=1.0
- joint thumb_cmc_roll: limit lower=0 upper=0.6108 effort=1 velocity=1 -> lower=0 upper=0.6311 effort=1 velocity=1; origin xyz=0.018722 0.016674 0.024272 rpy=0 0 0 -> xyz=0.018257 0.012998 0.024272 rpy=0 0 0
- joint thumb_cmc_yaw: limit lower=0 upper=1.63 effort=1 velocity=1 -> lower=0 upper=1.8718 effort=1 velocity=1; origin xyz=-0.00475 0.016238 -0.00059587 rpy=0 0 0 -> xyz=-0.00215 0.015238 0 rpy=0 0 0
- joint thumb_mcp: limit lower=0 upper=1.51 effort=1 velocity=1 -> lower=0 upper=1.8337 effort=1 velocity=1; origin xyz=-5.4077E-05 0.052039 0.0059395 rpy=0 0 0 -> xyz=0.00045 0.015539 0.0029937 rpy=-0.33161 0 0

Commit message: fix: finalize O30 hand models and LinkerForce configs

File: src/linkerhand_retarget/linkerhand_retarget/assets/robots/hands/linker_hand/o30_left/linkerhand_o30_left.urdf (robot description, URDF)
Before this commit: robot linkerhand_O30i_left.urdf, 21 links, 20 joints
Links:
- link hand_base_link: geometry collision mesh filename=meshes/hand_base_link.STL; visual mesh filename=meshes/hand_base_link.STL
- link index_distal: geometry collision mesh filename=meshes/index_distal.STL; visual mesh filename=meshes/index_distal.STL
- link index_metacarpals: geometry collision mesh filename=meshes/index_metacarpals.STL; visual mesh filename=meshes/index_metacarpals.STL
- link index_middle: geometry collision mesh filename=meshes/index_middle.STL; visual mesh filename=meshes/index_middle.STL
- link index_proximal: geometry collision mesh filename=meshes/index_proximal.STL; visual mesh filename=meshes/index_proximal.STL
- link middle_distal: geometry collision mesh filename=meshes/middle_distal.STL; visual mesh filename=meshes/middle_distal.STL
- link middle_metacarpals: geometry collision mesh filename=meshes/middle_metacarpals.STL; visual mesh filename=meshes/middle_metacarpals.STL
- link middle_middle: geometry collision mesh filename=meshes/middle_middle.STL; visual mesh filename=meshes/middle_middle.STL
- link middle_proximal: geometry collision mesh filename=meshes/middle_proximal.STL; visual mesh filename=meshes/middle_proximal.STL
- link pinky_distal: geometry collision mesh filename=meshes/pinky_distal.STL; visual mesh filename=meshes/pinky_distal.STL
- link pinky_metacarpals: geometry collision mesh filename=meshes/pinky_metacarpals.STL; visual mesh filename=meshes/pinky_metacarpals.STL
- link pinky_middle: geometry collision mesh filename=meshes/pinky_middle.STL; visual mesh filename=meshes/pinky_middle.STL
- link pinky_proximal: geometry collision mesh filename=meshes/pinky_proximal.STL; visual mesh filename=meshes/pinky_proximal.STL
- link ring_distal: geometry collision mesh filename=meshes/ring_distal.STL; visual mesh filename=meshes/ring_distal.STL
- link ring_metacarpals: geometry collision mesh filename=meshes/ring_metacarpals.STL; visual mesh filename=meshes/ring_metacarpals.STL
- link ring_middle: geometry collision mesh filename=meshes/ring_middle.STL; visual mesh filename=meshes/ring_middle.STL
- link ring_proximal: geometry collision mesh filename=meshes/ring_proximal.STL; visual mesh filename=meshes/ring_proximal.STL
- link thumb_distal: geometry collision mesh filename=meshes/thumb_distal.STL; visual mesh filename=meshes/thumb_distal.STL
- link thumb_metacarpals_base1: geometry collision mesh filename=meshes/thumb_metacarpals_base1.STL; visual mesh filename=meshes/thumb_metacarpals_base1.STL
- link thumb_metacarpals_base2: geometry collision mesh filename=meshes/thumb_metacarpals_base2.STL; visual mesh filename=meshes/thumb_metacarpals_base2.STL
- link thumb_proximal: geometry collision mesh filename=meshes/thumb_proximal.STL; visual mesh filename=meshes/thumb_proximal.STL
Joints:
- joint index_dip: axis 0.0 1.0 0.0 -> -0 1 -0; limit lower=0.0 upper=1.5967 effort=1.0 velocity=1.0 -> lower=0.0 upper=1.59669999534 effort=1.0 velocity=1.0; origin xyz=0.0 -0.0 0.040244 rpy=-0.0 -0.0 -0.0 -> xyz=0 -0 0.040244 rpy=-0 0.0402952773826 -0
- joint index_mcp_pitch: axis 0.0 1.0 0.0 -> -0 1 -0; limit lower=0.0 upper=1.8381 effort=1.0 velocity=1.0 -> lower=0.0 upper=1.735046222075943 effort=1.0 velocity=1.0; origin xyz=-0.00475 -0.00059587 0.016238 rpy=-0.0 -0.0 -0.0 -> xyz=-0.00475 -0.00059587 0.016238 rpy=-0 1.221245327087672e-14 -0
- joint index_mcp_roll: axis -1.0 -0.0 -0.0 -> -1 0 -0; limit lower=-0.397 upper=0.0203 effort=1.0 velocity=1.0 -> lower=-0.3970 upper=-0.0532672649819852 effort=1.0 velocity=1.0; origin xyz=0.018722 -0.029679 0.075158 rpy=-0.0 -0.0 -0.0 -> xyz=0.018722 -0.029679 0.075158 rpy=-0.05326726498196427 0 -0
- joint index_pip: axis 0.0 1.0 0.0 -> -0 1 -0; limit lower=0.0 upper=1.5958 effort=1.0 velocity=1.0 -> lower=0.0 upper=1.471362682698838 effort=1.0 velocity=1.0; origin xyz=0.0 -0.0 0.039681 rpy=-0.0 -0.0 -0.0 -> xyz=0 -0 0.039681 rpy=-0 -3.019806626980426e-14 -0
- joint middle_dip: axis 0.0 1.0 0.0 -> -0 1 -0; limit lower=0.0 upper=1.5851 effort=1.0 velocity=1.0 -> lower=0.0 upper=1.59776752134 effort=1.0 velocity=1.0; origin xyz=0.0 -0.0 0.040244 rpy=-0.0 -0.0 -0.0 -> xyz=0 -0 0.040244 rpy=-0 -0.0308518454734 -0
- joint middle_mcp_pitch: axis 0.0 1.0 0.0 -> -0 1 -0; limit lower=0.0 upper=1.8159 effort=1.0 velocity=1.0 -> lower=0.0 upper=1.586027117348012 effort=1.0 velocity=1.0; origin xyz=-0.00475 -0.00059587 0.016238 rpy=-0.0 -0.0 -0.0 -> xyz=-0.00475 -0.00059587 0.016238 rpy=-0 -0.01523079055311838 -0
- joint middle_mcp_roll: axis -1.0 -0.0 -0.0 -> -1 0 -0; limit lower=-0.4265 upper=0.1521 effort=1.0 velocity=1.0 -> lower=-0.4265 upper=0.1089663129860673 effort=1.0 velocity=1.0; origin xyz=0.018722 -0.0086937 0.081586 rpy=-0.0 -0.0 -0.0 -> xyz=0.018722 -0.0086937 0.08158600000000001 rpy=-0.0128260248695901 0 -0
- joint middle_pip: axis 0.0 1.0 0.0 -> -0 1 -0; limit lower=0.0 upper=1.5658 effort=1.0 velocity=1.0 -> lower=0.0 upper=1.590822001021158 effort=1.0 velocity=1.0; origin xyz=0.0 -0.0 0.039681 rpy=-0.0 -0.0 -0.0 -> xyz=0 -0 0.039681 rpy=-0 0.0138711925804 -0
- joint pinky_dip: axis 0.0 1.0 0.0 -> -0 1 -0; limit lower=0.0 upper=1.5897 effort=1.0 velocity=1.0 -> lower=0.0 upper=1.58606542135 effort=1.0 velocity=1.0; origin xyz=0.0 -0.0 0.040244 rpy=-0.0 -0.0 -0.0 -> xyz=0 -0 0.040244 rpy=-0 -0.0155350252509 -0
- joint pinky_mcp_pitch: axis 0.0 1.0 0.0 -> -0 1 -0; limit lower=0.0 upper=1.8241 effort=1.0 velocity=1.0 -> lower=0.0 upper=1.746158486401212 effort=1.0 velocity=1.0; origin xyz=-0.00475 -0.00059587 0.016238 rpy=-0.0 -0.0 -0.0 -> xyz=-0.00475 -0.00059587 0.016238 rpy=-0 -0.0220425694976 -0
- joint pinky_mcp_roll: axis -1.0 -0.0 -0.0 -> -1 0 -0; limit lower=-0.0548 upper=0.3874 effort=1.0 velocity=1.0 -> lower=-0.0548 upper=0.3102413287225498 effort=1.0 velocity=1.0; origin xyz=0.018722 0.030927 0.067761 rpy=-0.0 -0.0 -0.0 -> xyz=0.018722 0.030927 0.067761 rpy=-0.01471703057163711 0 -0
- joint pinky_pip: axis 0.0 1.0 0.0 -> -0 1 -0; limit lower=0.0 upper=1.5123 effort=1.0 velocity=1.0 -> lower=0.0 upper=1.57669319439 effort=1.0 velocity=1.0; origin xyz=0.0 -0.0 0.039681 rpy=-0.0 -0.0 -0.0 -> xyz=0 -0 0.039681 rpy=-0 0.0153062751135 -0
- joint ring_dip: axis 0.0 1.0 0.0 -> -0 1 -0; limit lower=0.0 upper=1.5391 effort=1.0 velocity=1.0 -> lower=0.0 upper=1.5742161012 effort=1.0 velocity=1.0; origin xyz=0.0 -0.0 0.040244 rpy=-0.0 -0.0 -0.0 -> xyz=0 -0 0.040244 rpy=-0 -0.00428430308889 -0
- joint ring_mcp_pitch: axis 0.0 1.0 0.0 -> -0 1 -0; limit lower=0.0 upper=1.8145 effort=1.0 velocity=1.0 -> lower=0.0 upper=1.55394971023 effort=1.0 velocity=1.0; origin xyz=-0.00475 -0.00059587 0.016238 rpy=-0.0 -0.0 -0.0 -> xyz=-0.00475 -0.00059587 0.016238 rpy=-0 0.0255589602002 -0
- joint ring_mcp_roll: axis -1.0 -0.0 -0.0 -> -1 0 -0; limit lower=-0.2288 upper=0.3049 effort=0.0 velocity=0.0 -> lower=-0.2288 upper=0.2882392053656797 effort=0.0 velocity=0.0; origin xyz=0.018722 0.012188 0.079218 rpy=-0.0 -0.0 -0.0 -> xyz=0.018722 0.012188 0.079218 rpy=-0.005763480038315312 0 -0
- joint ring_pip: axis 0.0 1.0 0.0 -> -0 1 -0; limit lower=0.0 upper=1.4911 effort=1.0 velocity=1.0 -> lower=0.0 upper=1.58679961547 effort=1.0 velocity=1.0; origin xyz=0.0 -0.0 0.039681 rpy=-0.0 -0.0 -0.0 -> xyz=0 -0 0.039681 rpy=-0 0.0220509528547 -0
- joint thumb_cmc_roll: axis -1.0 -0.0 -0.0 -> -1 0 -0; limit lower=0.0 upper=0.6311 effort=1.0 velocity=1.0 -> lower=0 upper=0.87226588169 effort=1 velocity=1; origin xyz=0.018257 -0.012998 0.024272 rpy=-0.0 -0.0 -0.0 -> xyz=0.018257 -0.012998 0.024272 rpy=0.07680614007600001 0 -0
- joint thumb_cmc_yaw: axis -0.0 -0.0 1.0 -> -0 0 1; limit lower=0.0 upper=1.8718 effort=1.0 velocity=1.0 -> lower=0 upper=2.02824782456 effort=1 velocity=1; origin xyz=-0.00215 -0.015238 0.0 rpy=-0.0 -0.0 -0.0 -> xyz=-0.00215 -0.015238 0 rpy=-0 0 0.0283606787672
- joint thumb_ip: axis -1.0 -0.0 -0.0 -> -1 0 -0; limit lower=0.0 upper=1.5912 effort=1.0 velocity=1.0 -> lower=0 upper=1.603532956380333 effort=1 velocity=1; origin xyz=0.0 -0.048532 0.00155 rpy=-0.0 -0.0 -0.0 -> xyz=0 -0.048532 0.00155 rpy=0.0327366295854 0 -0
- joint thumb_mcp: axis -1.0 -0.0 -0.0 -> -1 0 -0; limit lower=0.0 upper=1.8337 effort=1.0 velocity=1.0 -> lower=0 upper=1.9412774217 effort=1 velocity=1; origin xyz=0.00045 -0.015539 0.0029937 rpy=0.33161 -0.0 -0.0 -> xyz=0.00045 -0.015539 0.0029937 rpy=0.384266722602 0 -0

File: src/linkerhand_retarget/linkerhand_retarget/assets/robots/hands/linker_hand/o30_right/linkerhand_o30_right.urdf (robot description, URDF)
Before this commit: robot linkerhand_O30i_right.urdf, 21 links, 20 joints
Joints:
- joint index_dip: limit lower=0.0 upper=1.5967 effort=1.0 velocity=1.0 -> lower=0.0 upper=1.59669999534 effort=1.0 velocity=1.0; origin xyz=0 0 0.040244 rpy=0 0 0 -> xyz=0 0 0.040244 rpy=0 0.0402952773826 0
- joint index_mcp_pitch: limit lower=0.0 upper=1.8381 effort=1.0 velocity=1.0 -> lower=0.0 upper=1.735046222075943 effort=1.0 velocity=1.0; origin xyz=-0.00475 0.00059587 0.016238 rpy=0 0 0 -> xyz=-0.00475 0.00059587 0.016238 rpy=0 1.221245327087672e-14 0
- joint index_mcp_roll: limit lower=-0.3970 upper=0.0203 effort=1.0 velocity=1.0 -> lower=-0.3970 upper=-0.0532672649819852 effort=1.0 velocity=1.0; origin xyz=0.018722 0.029679 0.075158 rpy=0 0 0 -> xyz=0.018722 0.029679 0.075158 rpy=0.05326726498196427 0 0
- joint index_pip: limit lower=0.0 upper=1.5958 effort=1.0 velocity=1.0 -> lower=0.0 upper=1.471362682698838 effort=1.0 velocity=1.0; origin xyz=0 0 0.039681 rpy=0 0 0 -> xyz=0 0 0.039681 rpy=0 -3.019806626980426e-14 0
- joint middle_dip: limit lower=0.0 upper=1.5851 effort=1.0 velocity=1.0 -> lower=0.0 upper=1.59776752134 effort=1.0 velocity=1.0; origin xyz=0 0 0.040244 rpy=0 0 0 -> xyz=0 0 0.040244 rpy=0 -0.0308518454734 0
- joint middle_mcp_pitch: limit lower=0.0 upper=1.8159 effort=1.0 velocity=1.0 -> lower=0.0 upper=1.586027117348012 effort=1.0 velocity=1.0; origin xyz=-0.00475 0.00059587 0.016238 rpy=0 0 0 -> xyz=-0.00475 0.00059587 0.016238 rpy=0 -0.01523079055311838 0
- joint middle_mcp_roll: limit lower=-0.4265 upper=0.1521 effort=1.0 velocity=1.0 -> lower=-0.4265 upper=0.1089663129860673 effort=1.0 velocity=1.0; origin xyz=0.018722 0.0086937 0.081586 rpy=0 0 0 -> xyz=0.018722 0.0086937 0.081586 rpy=0.0128260248695901 0 0
- joint middle_pip: limit lower=0.0 upper=1.5658 effort=1.0 velocity=1.0 -> lower=0.0 upper=1.590822001021158 effort=1.0 velocity=1.0; origin xyz=0 0 0.039681 rpy=0 0 0 -> xyz=0 0 0.039681 rpy=0 0.0138711925804 0
- joint pinky_dip: limit lower=0.0 upper=1.5897 effort=1.0 velocity=1.0 -> lower=0.0 upper=1.58606542135 effort=1.0 velocity=1.0; origin xyz=0 0 0.040244 rpy=0 0 0 -> xyz=0 0 0.040244 rpy=0 -0.0155350252509 0
- joint pinky_mcp_pitch: limit lower=0.0 upper=1.8241 effort=1.0 velocity=1.0 -> lower=0.0 upper=1.746158486401212 effort=1.0 velocity=1.0; origin xyz=-0.00475 0.00059587 0.016238 rpy=0 0 0 -> xyz=-0.00475 0.00059587 0.016238 rpy=0 -0.0220425694976 0
- joint pinky_mcp_roll: limit lower=-0.0548 upper=0.3874 effort=1.0 velocity=1.0 -> lower=-0.0548 upper=0.3102413287225498 effort=1.0 velocity=1.0; origin xyz=0.018722 -0.030927 0.067761 rpy=0 0 0 -> xyz=0.018722 -0.030927 0.067761 rpy=0.01471703057163711 0 0
- joint pinky_pip: limit lower=0.0 upper=1.5123 effort=1.0 velocity=1.0 -> lower=0.0 upper=1.57669319439 effort=1.0 velocity=1.0; origin xyz=0 0 0.039681 rpy=0 0 0 -> xyz=0 0 0.039681 rpy=0 0.0153062751135 0
- joint ring_dip: limit lower=0.0 upper=1.5391 effort=1.0 velocity=1.0 -> lower=0.0 upper=1.5742161012 effort=1.0 velocity=1.0; origin xyz=0 0 0.040244 rpy=0 0 0 -> xyz=0 0 0.040244 rpy=0 -0.00428430308889 0
- joint ring_mcp_pitch: limit lower=0.0 upper=1.8145 effort=1.0 velocity=1.0 -> lower=0.0 upper=1.55394971023 effort=1.0 velocity=1.0; origin xyz=-0.00475 0.00059587 0.016238 rpy=0 0 0 -> xyz=-0.00475 0.00059587 0.016238 rpy=0 0.0255589602002 0
- joint ring_mcp_roll: limit lower=-0.2288 upper=0.3049 effort=0.0 velocity=0.0 -> lower=-0.2288 upper=0.2882392053656797 effort=0.0 velocity=0.0; origin xyz=0.018722 -0.012188 0.079218 rpy=0 0 0 -> xyz=0.018722 -0.012188 0.079218 rpy=0.005763480038315312 0 0
- joint ring_pip: limit lower=0.0 upper=1.4911 effort=1.0 velocity=1.0 -> lower=0.0 upper=1.58679961547 effort=1.0 velocity=1.0; origin xyz=0 0 0.039681 rpy=0 0 0 -> xyz=0 0 0.039681 rpy=0 0.0220509528547 0
- joint thumb_cmc_roll: limit lower=0 upper=0.6311 effort=1 velocity=1 -> lower=0 upper=0.87226588169 effort=1 velocity=1; origin xyz=0.018257 0.012998 0.024272 rpy=0 0 0 -> xyz=0.018257 0.012998 0.024272 rpy=-0.076806140076 0 0
- joint thumb_cmc_yaw: limit lower=0 upper=1.8718 effort=1 velocity=1 -> lower=0 upper=2.02824782456 effort=1 velocity=1; origin xyz=-0.00215 0.015238 0 rpy=0 0 0 -> xyz=-0.00215 0.015238 0 rpy=0 0 -0.0283606787672
- joint thumb_ip: limit lower=0 upper=1.5912 effort=1 velocity=1 -> lower=0 upper=1.603532956380333 effort=1 velocity=1; origin xyz=0 0.048532 0.00155 rpy=0 0 0 -> xyz=0 0.048532 0.00155 rpy=-0.0327366295854 0 0
- joint thumb_mcp: limit lower=0 upper=1.8337 effort=1 velocity=1 -> lower=0 upper=1.9412774217 effort=1 velocity=1; origin xyz=0.00045 0.015539 0.0029937 rpy=-0.33161 0 0 -> xyz=0.00045 0.015539 0.0029937 rpy=-0.384266722602 0 0
